Commit message: Added a low poly version of the mogabot2 stl files

File: mogabot2_description/urdf/mogabot2.urdf.xacro (robot description, xacro)
@@ -5,5 +5,5 @@
         <visual>
             <geometry>
-                <mesh filename="package://mogabot2_description/meshes/1_World_to_base.stl"
+                <mesh filename="package://mogabot2_description/meshes/1_World_to_base_lowpoly.stl"
                       scale="0.01 0.01 0.01"/>
             </geometry>
@@ -12,5 +12,5 @@
         <collision>
             <geometry>
-                <mesh filename="package://mogabot2_description/meshes/1_World_to_base.stl"
+                <mesh filename="package://mogabot2_description/meshes/1_World_to_base_lowpoly.stl"
                       scale="0.01 0.01 0.01"/>
             </geometry>
@@ -21,5 +21,5 @@
         <visual>
             <geometry>
-                <mesh filename="package://mogabot2_description/meshes/2_Base_to_Shoulder.stl"
+                <mesh filename="package://mogabot2_description/meshes/2_Base_to_Shoulder_lowpoly.stl"
                       scale="0.01 0.01 0.01"/>
             </geometry>
@@ -28,5 +28,5 @@
         <collision>
             <geometry>
-                <mesh filename="package://mogabot2_description/meshes/2_Base_to_Shoulder.stl"
+                <mesh filename="package://mogabot2_description/meshes/2_Base_to_Shoulder_lowpoly.stl"
                       scale="0.01 0.01 0.01"/>
             </geometry>
@@ -37,5 +37,5 @@
         <visual>
             <geometry>
-                <mesh filename="package://mogabot2_description/meshes/3_Shoulder_to_Elbow.stl"
+                <mesh filename="package://mogabot2_description/meshes/3_Shoulder_to_Elbow_lowpoly.stl"
                       scale="0.01 0.01 0.01"/>
             </geometry>
@@ -44,5 +44,5 @@
         <collision>
             <geometry>
-                <mesh filename="package://mogabot2_description/meshes/3_Shoulder_to_Elbow.stl"
+                <mesh filename="package://mogabot2_description/meshes/3_Shoulder_to_Elbow_lowpoly.stl"
                       scale="0.01 0.01 0.01"/>
             </geometry>
@@ -53,5 +53,5 @@
         <visual>
             <geometry>
-                <mesh filename="package://mogabot2_description/meshes/4_Elbow_to_Forarm_bis.stl"
+                <mesh filename="package://mogabot2_description/meshes/4_Elbow_to_Forarm_bis_lowpoly.stl"
                       scale="0.01 0.01 0.01"/>
             </geometry>
@@ -60,5 +60,5 @@
         <collision>
             <geometry>
-                <mesh filename="package://mogabot2_description/meshes/4_Elbow_to_Forarm_bis.stl"
+                <mesh filename="package://mogabot2_description/meshes/4_Elbow_to_Forarm_bis_lowpoly.stl"
                       scale="0.01 0.01 0.01"/>
             </geometry>
@@ -69,5 +69,5 @@
         <visual>
             <geometry>
-                <mesh filename="package://mogabot2_description/meshes/5_Forarm_to_Wrist.stl"
+                <mesh filename="package://mogabot2_description/meshes/5_Forarm_to_Wrist_lowpoly.stl"
                       scale="0.01 0.01 0.01"/>
             </geometry>
@@ -76,5 +76,5 @@
         <collision>
             <geometry>
-                <mesh filename="package://mogabot2_description/meshes/5_Forarm_to_Wrist.stl"
+                <mesh filename="package://mogabot2_description/meshes/5_Forarm_to_Wrist_lowpoly.stl"
                       scale="0.01 0.01 0.01"/>
             </geometry>
@@ -85,5 +85,5 @@
         <visual>
             <geometry>
-                <mesh filename="package://mogabot2_description/meshes/6_Wrist_to_Hand.stl"
+                <mesh filename="package://mogabot2_description/meshes/6_Wrist_to_Hand_lowpoly.stl"
                       scale="0.01 0.01 0.01"/>
             </geometry>
@@ -92,5 +92,5 @@
         <collision>
             <geometry>
-                <mesh filename="package://mogabot2_description/meshes/6_Wrist_to_Hand.stl"
+                <mesh filename="package://mogabot2_description/meshes/6_Wrist_to_Hand_lowpoly.stl"
                       scale="0.01 0.01 0.01"/>
             </geometry>
@@ -101,5 +101,5 @@
         <visual>
             <geometry>
-                <mesh filename="package://mogabot2_description/meshes/7_Hand_to_Gripper.stl"
+                <mesh filename="package://mogabot2_description/meshes/7_Hand_to_Gripper_lowpoly.stl"
                       scale="0.01 0.01 0.01"/>
             </geometry>
@@ -108,5 +108,5 @@
         <collision>
             <geometry>
-                <mesh filename="package://mogabot2_description/meshes/7_Hand_to_Gripper.stl"
+                <mesh filename="package://mogabot2_description/meshes/7_Hand_to_Gripper_lowpoly.stl"
                       scale="0.01 0.01 0.01"/>
             </geometry>

Commit message: Set up path planning with visualization for mogabot2 robot - collisions not managed

File: mogabot2_description/urdf/mogabot2.urdf.xacro (robot description, xacro)
@@ -10,11 +10,4 @@
             <origin xyz="0 0 0" rpy="0 0 0"/>
         </visual>
-        <collision>
-            <geometry>
-                <mesh filename="package://mogabot2_description/meshes/1_World_to_base_lowpoly.stl"
-                      scale="0.01 0.01 0.01"/>
-            </geometry>
-            <origin xyz="0 0 0" rpy="0 0 0"/>
-        </collision>
     </link>
     <link name="shoulder_link">
@@ -26,11 +19,4 @@
             <origin xyz="0 0 0" rpy="0 0 0"/>
         </visual>
-        <collision>
-            <geometry>
-                <mesh filename="package://mogabot2_description/meshes/2_Base_to_Shoulder_lowpoly.stl"
-                      scale="0.01 0.01 0.01"/>
-            </geometry>
-            <origin xyz="0 0 0" rpy="0 0 0"/>
-        </collision>
     </link>
     <link name="arm1_link">
@@ -42,11 +28,4 @@
             <origin xyz="0 0 0" rpy="0 0 0"/>
         </visual>
-        <collision>
-            <geometry>
-                <mesh filename="package://mogabot2_description/meshes/3_Shoulder_to_Elbow_lowpoly.stl"
-                      scale="0.01 0.01 0.01"/>
-            </geometry>
-            <origin xyz="0 0 0" rpy="0 0 0"/>
-        </collision>
     </link>
     <link name="elbow_link">
@@ -58,11 +37,4 @@
             <origin xyz="0 0 0" rpy="0 0 3.14"/>
         </visual>
-        <collision>
-            <geometry>
-                <mesh filename="package://mogabot2_description/meshes/4_Elbow_to_Forarm_bis_lowpoly.stl"
-                      scale="0.01 0.01 0.01"/>
-            </geometry>
-            <origin xyz="0 0 0" rpy="0 0 3.14"/>
-        </collision>
     </link>
     <link name="forarm_link">
@@ -74,11 +46,4 @@
             <origin xyz="0 0 0" rpy="3.14 3.14 0"/>
         </visual>
-        <collision>
-            <geometry>
-                <mesh filename="package://mogabot2_description/meshes/5_Forarm_to_Wrist_lowpoly.stl"
-                      scale="0.01 0.01 0.01"/>
-            </geometry>
-            <origin xyz="0 0 0" rpy="3.14 3.14 0"/>
-        </collision>
     </link>
     <link name="wrist_link">
@@ -90,11 +55,4 @@
             <origin xyz="0 0 0" rpy="3.14 3.14 0"/>
         </visual>
-        <collision>
-            <geometry>
-                <mesh filename="package://mogabot2_description/meshes/6_Wrist_to_Hand_lowpoly.stl"
-                      scale="0.01 0.01 0.01"/>
-            </geometry>
-            <origin xyz="0 0 0" rpy="3.14 3.14 0"/>
-        </collision>
     </link>
     <link name="hand_link">
@@ -106,11 +64,4 @@
             <origin xyz="0 -0.2 0" rpy="3.14 0 0"/>
         </visual>
-        <collision>
-            <geometry>
-                <mesh filename="package://mogabot2_description/meshes/7_Hand_to_Gripper_lowpoly.stl"
-                      scale="0.01 0.01 0.01"/>
-            </geometry>
-            <origin xyz="0 0 0" rpy="3.14 0 0"/>
-        </collision>
     </link>
 <!--
